File: Wersja 2.0/course_boards.kicad_sch (KiCad schematic)
At the start: 33 parts, among them J1 POWER_SOCKET, J2 Conn_01x02_Socket, J3 Conn_01x02_Socket, Q1 BC547, Q3 BC547, SW1 SW_Push, SW2 SW_Push, SW3 SW_Push, U1 ESP32-C3-DevKitM-1

Commit message: fix ver 2
Parts:
- removed J2, J3: Conn_01x02_Socket, symbol Connector:Conn_01x02_Socket
- removed U1: ESP32-C3-DevKitM-1, RF_Module:ESP32-C3-DevKitM-1, symbol RF_Module:ESP32-C3-DevKitM-1
- added J2: I2C_CONN, Connector_PinHeader_2.54mm:PinHeader_1x04_P2.54mm_Vertical, symbol Connector_Generic:Conn_01x04
- added J4: UART_CONN, Connector_PinHeader_2.54mm:PinHeader_1x04_P2.54mm_Vertical, symbol Connector_Generic:Conn_01x04
- added U1: ESP32-C6-DevKitC-1, PCM_Espressif:ESP32-C6-DevKitC-1, symbol PCM_Espressif:ESP32-C6-DevKitC-1
Connections:
- net GND: now also J2.1 (Pin_1), J4.1 (Pin_1), U1.15 (GND), U1.18 (GND), U1.21 (GND), U1.32 (GND)
- net VCC: now also U1.14 (5V); no longer RV5K1.1
- net at RV5K1.2: now also U1.3 (GPIO4/MTMS)
- net at R4.1: now also U1.12 (GPIO2)
- net at R7.1: now also U1.13 (GPIO3)
- new net: J4.2 (Pin_2), U1.8 (GPIO1)
- new net: J4.3 (Pin_3), U1.7 (GPIO0)
- new net: J2.2 (Pin_2), U1.4 (GPIO5/MTDI)
- new net: J2.3 (Pin_3), U1.5 (GPIO6)
- new net 3V3: J2.4 (Pin_4), J4.4 (Pin_4), RV5K1.1, U1.1 (3V3)
- no-connect marks 0 -> 19
Other:
- moved on the sheet: D10, D3, R4, R7, RV5K1
