File: Wersja 2.0/course_boards.kicad_pcb (KiCad board)
At the start: 2 copper layers, 167.5 x 83.8 mm, 72 parts, among them J1 POWER_SOCKET, J2 I2C_CONN, J4 UART_CONN, Q1 BC547, Q3 BC547, SW1 SW_Push, SW2 SW_Push, SW3 SW_Push, U1 ESP32-C6-DevKitC-1

Commit message: fix typo
Other:
- board text added: "AIOTA X AGH Drone Engineering X Logic_Laboratory"
- board text removed: "AIOTA X AGH Drone Engineering X Logic_Labolatory"
Changed lines of the file:
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@@
 		)
 	)
-	(gr_text "AIOTA X AGH Drone Engineering X Logic_Labolatory"
+	(gr_text "AIOTA X AGH Drone Engineering X Logic_Laboratory"
 		(at 76.3 84.455 0)
 		(layer "F.SilkS")

Commit message: v2.3
Parts:
- moved RV5KK1 0.71 mm to (67.6, 50.8)
Changed lines of the file:
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@@
 	(footprint "Potentiometer_THT:Potentiometer_Alps_RK163_Single_Horizontal"
 		(layer "F.Cu")
-		(at 67.5 51.5)
+		(at 67.6 50.8)
 		(descr "1110U1Q 1110TNP 1110U2A 1110U0Q Potentiometer, horizontal, Alps RK163 Single, https://tech.alpsalpine.com/prod/e/pdf/potentiometer/rotarypotentiometers/rk16/rk16.pdf")
 		(tags "Potentiometer horizontal Alps RK163 Single")
@@
 	)
 	(gr_rect
-		(start 55.6 52.4)
-		(end 58.3 60.7)
+		(start 55.6 51.75)
+		(end 58.3 60.05)
 		(stroke
 			(width 0.1)
@@
 	)
 	(gr_line
-		(start 56.95 52.4)
+		(start 56.95 51.75)
 		(end 56.95 51.75)
 		(stroke
@@
 	(gr_line
 		(start 56.95 62)
-		(end 56.95 60.7)
+		(end 56.95 60.05)
 		(stroke
 			(width 0.1)
@@
 	)
 	(segment
-		(start 67.4525 51.35)
-		(end 71.9 46.9025)
+		(start 151.25 82.905)
+		(end 149.78 84.375)
 		(width 2)
 		(layer "B.Cu")
@@
 	)
 	(segment
-		(start 151.25 82.905)
-		(end 149.78 84.375)
+		(start 67.6 50.8)
+		(end 68.0025 50.8)
 		(width 2)
 		(layer "B.Cu")
@@
 	)
 	(segment
+		(start 68.0025 50.8)
+		(end 71.9 46.9025)
+		(width 2)
+		(layer "B.Cu")
+		(net 5)
+	)
+	(segment
 		(start 70.485 90.17)
 		(end 68.1 90.17)
@@
 		(width 2)
 		(layer "B.Cu")
-		(net 5)
-	)
-	(segment
-		(start 67.45 51.35)
-		(end 67.4525 51.35)
-		(width 2)
-		(layer "B.Cu")

Commit message: more pads!
Parts:
- added ?: , , F.Cu at (200.4, 125.4)
- added ?: , , F.Cu at (205.4, 119.9)
- added ?: , , F.Cu at (200.4, 119.9)
- added ?: , , F.Cu at (205.4, 125.4)
- moved ? 9.56 mm to (196.0, 123.8)
- moved ? 9.56 mm to (185.8, 120.2)
- moved ? 9.56 mm to (190.9, 120.2)
- moved ? 9.56 mm to (178.2, 123.8)
- moved ? 9.56 mm to (185.8, 123.8)
- moved ? 9.56 mm to (180.7, 120.2)
- moved ? 9.56 mm to (188.3, 123.8)
- moved ? 9.56 mm to (188.3, 120.2)
- moved ? 9.56 mm to (190.9, 123.8)
- moved ? 9.56 mm to (183.3, 120.2)
- moved ? 9.56 mm to (178.2, 120.2)
- moved ? 9.56 mm to (193.4, 120.2)
- moved ? 9.56 mm to (183.3, 123.8)
- moved ? 9.56 mm to (196.0, 120.2)
- moved ? 9.56 mm to (193.4, 123.8)
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